Commit message: base fixed to the world 0 0 0

File: src/mecademic_description/urdf/meca_500_r3.urdf.xacro (robot description, xacro)
@@ -1,3 +1,15 @@
 <?xml version="1.0" encoding="utf-8" ?>
+<!-- =================================================================================== -->
+<!-- |    This document was autogenerated by xacro from /home/ram/Projects/Project-Interstellar/src/mecademic_description/urdf/meca_500_r3.urdf.xacro | -->
+<!-- |    EDITING THIS FILE BY HAND IS NOT RECOMMENDED                                 | -->
+<!-- =================================================================================== -->
+<!-- =================================================================================== -->
+<!-- |    This document was autogenerated by xacro from /home/ram/Projects/Project-Interstellar/src/mecademic_description/urdf/meca_500_r3.urdf.xacro | -->
+<!-- |    EDITING THIS FILE BY HAND IS NOT RECOMMENDED                                 | -->
+<!-- =================================================================================== -->
+<!-- =================================================================================== -->
+<!-- |    This document was autogenerated by xacro from /home/ram/Projects/Project-Interstellar/src/mecademic_description/urdf/meca_500_r3.urdf.xacro | -->
+<!-- |    EDITING THIS FILE BY HAND IS NOT RECOMMENDED                                 | -->
+<!-- =================================================================================== -->
 <!-- =================================================================================== -->
 <!-- |    This document was autogenerated by xacro from /home/ram/ws_moveit/src/mecademic_description/urdf/meca_500_r3.urdf.xacro | -->
@@ -9,4 +21,9 @@
 <!-- =================================================================================== -->
 <robot name="meca_500_r3">
+    <link name="world"/>
+    <joint name="fixed" type="fixed">
+        <parent link="world"/>
+        <child link="meca_base_link"/>
+    </joint>
     <!-- Base link is the center of the robot's bottom plate -->
     <link name="meca_base_link">
@@ -310,4 +327,199 @@
     </transmission>
     <gazebo>
+        <plugin filename="libgazebo_ros_control.so" name="gazebo_ros_control">
+            <robotNamespace>/</robotNamespace>
+        </plugin>
+    </gazebo>
+    <transmission name="trans_meca_axis_1_joint">
+        <type>transmission_interface/SimpleTransmission</type>
+        <joint name="meca_axis_1_joint">
+            <hardwareInterface>hardware_interface/EffortJointInterface</hardwareInterface>
+        </joint>
+        <actuator name="meca_axis_1_joint_motor">
+            <hardwareInterface>hardware_interface/EffortJointInterface</hardwareInterface>
+            <mechanicalReduction>1</mechanicalReduction>
+        </actuator>
+    </transmission>
+    <transmission name="trans_meca_axis_2_joint">
+        <type>transmission_interface/SimpleTransmission</type>
+        <joint name="meca_axis_2_joint">
+            <hardwareInterface>hardware_interface/EffortJointInterface</hardwareInterface>
+        </joint>
+        <actuator name="meca_axis_2_joint_motor">
+            <hardwareInterface>hardware_interface/EffortJointInterface</hardwareInterface>
+            <mechanicalReduction>1</mechanicalReduction>
+        </actuator>
+    </transmission>
+    <transmission name="trans_meca_axis_3_joint">
+        <type>transmission_interface/SimpleTransmission</type>
+        <joint name="meca_axis_3_joint">
+            <hardwareInterface>hardware_interface/EffortJointInterface</hardwareInterface>
+        </joint>
+        <actuator name="meca_axis_3_joint_motor">
+            <hardwareInterface>hardware_interface/EffortJointInterface</hardwareInterface>
+            <mechanicalReduction>1</mechanicalReduction>
+        </actuator>
+    </transmission>
+    <transmission name="trans_meca_axis_4_joint">
+        <type>transmission_interface/SimpleTransmission</type>
+        <joint name="meca_axis_4_joint">
+            <hardwareInterface>hardware_interface/EffortJointInterface</hardwareInterface>
+        </joint>
+        <actuator name="meca_axis_4_joint_motor">
+            <hardwareInterface>hardware_interface/EffortJointInterface</hardwareInterface>
+            <mechanicalReduction>1</mechanicalReduction>
+        </actuator>
+    </transmission>
+    <transmission name="trans_meca_axis_5_joint">
+        <type>transmission_interface/SimpleTransmission</type>
+        <joint name="meca_axis_5_joint">
+            <hardwareInterface>hardware_interface/EffortJointInterface</hardwareInterface>
+        </joint>
+        <actuator name="meca_axis_5_joint_motor">
+            <hardwareInterface>hardware_interface/EffortJointInterface</hardwareInterface>
+            <mechanicalReduction>1</mechanicalReduction>
+        </actuator>
+    </transmission>
+    <transmission name="trans_meca_axis_6_joint">
+        <type>transmission_interface/SimpleTransmission</type>
+        <joint name="meca_axis_6_joint">
+            <hardwareInterface>hardware_interface/EffortJointInterface</hardwareInterface>
+        </joint>
+        <actuator name="meca_axis_6_joint_motor">
+            <hardwareInterface>hardware_interface/EffortJointInterface</hardwareInterface>
+            <mechanicalReduction>1</mechanicalReduction>
+        </actuator>
+    </transmission>
+    <gazebo>
+        <plugin filename="libgazebo_ros_control.so" name="gazebo_ros_control">
+            <robotNamespace>/</robotNamespace>
+        </plugin>
+    </gazebo>
+    <transmission name="trans_meca_axis_1_joint">
+        <type>transmission_interface/SimpleTransmission</type>
+        <joint name="meca_axis_1_joint">
+            <hardwareInterface>hardware_interface/EffortJointInterface</hardwareInterface>
+        </joint>
+        <actuator name="meca_axis_1_joint_motor">
+            <hardwareInterface>hardware_interface/EffortJointInterface</hardwareInterface>
+            <mechanicalReduction>1</mechanicalReduction>
+        </actuator>
+    </transmission>
+    <transmission name="trans_meca_axis_2_joint">
+        <type>transmission_interface/SimpleTransmission</type>
+        <joint name="meca_axis_2_joint">
+            <hardwareInterface>hardware_interface/EffortJointInterface</hardwareInterface>
+        </joint>
+        <actuator name="meca_axis_2_joint_motor">
+            <hardwareInterface>hardware_interface/EffortJointInterface</hardwareInterface>
+            <mechanicalReduction>1</mechanicalReduction>
+        </actuator>
+    </transmission>
+    <transmission name="trans_meca_axis_3_joint">
+        <type>transmission_interface/SimpleTransmission</type>
+        <joint name="meca_axis_3_joint">
+            <hardwareInterface>hardware_interface/EffortJointInterface</hardwareInterface>
+        </joint>
+        <actuator name="meca_axis_3_joint_motor">
+            <hardwareInterface>hardware_interface/EffortJointInterface</hardwareInterface>
+            <mechanicalReduction>1</mechanicalReduction>
+        </actuator>
+    </transmission>
+    <transmission name="trans_meca_axis_4_joint">
+        <type>transmission_interface/SimpleTransmission</type>
+        <joint name="meca_axis_4_joint">
+            <hardwareInterface>hardware_interface/EffortJointInterface</hardwareInterface>
+        </joint>
+        <actuator name="meca_axis_4_joint_motor">
+            <hardwareInterface>hardware_interface/EffortJointInterface</hardwareInterface>
+            <mechanicalReduction>1</mechanicalReduction>
+        </actuator>
+    </transmission>
+    <transmission name="trans_meca_axis_5_joint">
+        <type>transmission_interface/SimpleTransmission</type>
+        <joint name="meca_axis_5_joint">
+            <hardwareInterface>hardware_interface/EffortJointInterface</hardwareInterface>
+        </joint>
+        <actuator name="meca_axis_5_joint_motor">
+            <hardwareInterface>hardware_interface/EffortJointInterface</hardwareInterface>
+            <mechanicalReduction>1</mechanicalReduction>
+        </actuator>
+    </transmission>
+    <transmission name="trans_meca_axis_6_joint">
+        <type>transmission_interface/SimpleTransmission</type>
+        <joint name="meca_axis_6_joint">
+            <hardwareInterface>hardware_interface/EffortJointInterface</hardwareInterface>
+        </joint>
+        <actuator name="meca_axis_6_joint_motor">
+            <hardwareInterface>hardware_interface/EffortJointInterface</hardwareInterface>
+            <mechanicalReduction>1</mechanicalReduction>
+        </actuator>
+    </transmission>
+    <gazebo>
+        <plugin filename="libgazebo_ros_control.so" name="gazebo_ros_control">
+            <robotNamespace>/</robotNamespace>
+        </plugin>
+    </gazebo>
+    <transmission name="trans_meca_axis_1_joint">
+        <type>transmission_interface/SimpleTransmission</type>
+        <joint name="meca_axis_1_joint">
+            <hardwareInterface>hardware_interface/EffortJointInterface</hardwareInterface>
+        </joint>
+        <actuator name="meca_axis_1_joint_motor">
+            <hardwareInterface>hardware_interface/EffortJointInterface</hardwareInterface>
+            <mechanicalReduction>1</mechanicalReduction>
+        </actuator>
+    </transmission>
+    <transmission name="trans_meca_axis_2_joint">
+        <type>transmission_interface/SimpleTransmission</type>
+        <joint name="meca_axis_2_joint">
+            <hardwareInterface>hardware_interface/EffortJointInterface</hardwareInterface>
+        </joint>
+        <actuator name="meca_axis_2_joint_motor">
+            <hardwareInterface>hardware_interface/EffortJointInterface</hardwareInterface>
+            <mechanicalReduction>1</mechanicalReduction>
+        </actuator>
+    </transmission>
+    <transmission name="trans_meca_axis_3_joint">
+        <type>transmission_interface/SimpleTransmission</type>
+        <joint name="meca_axis_3_joint">
+            <hardwareInterface>hardware_interface/EffortJointInterface</hardwareInterface>
+        </joint>
+        <actuator name="meca_axis_3_joint_motor">
+            <hardwareInterface>hardware_interface/EffortJointInterface</hardwareInterface>
+            <mechanicalReduction>1</mechanicalReduction>
+        </actuator>
+    </transmission>
+    <transmission name="trans_meca_axis_4_joint">
+        <type>transmission_interface/SimpleTransmission</type>
+        <joint name="meca_axis_4_joint">
+            <hardwareInterface>hardware_interface/EffortJointInterface</hardwareInterface>
+        </joint>
+        <actuator name="meca_axis_4_joint_motor">
+            <hardwareInterface>hardware_interface/EffortJointInterface</hardwareInterface>
+            <mechanicalReduction>1</mechanicalReduction>
+        </actuator>
+    </transmission>
+    <transmission name="trans_meca_axis_5_joint">
+        <type>transmission_interface/SimpleTransmission</type>
+        <joint name="meca_axis_5_joint">
+            <hardwareInterface>hardware_interface/EffortJointInterface</hardwareInterface>
+        </joint>
+        <actuator name="meca_axis_5_joint_motor">
+            <hardwareInterface>hardware_interface/EffortJointInterface</hardwareInterface>
+            <mechanicalReduction>1</mechanicalReduction>
+        </actuator>
+    </transmission>
+    <transmission name="trans_meca_axis_6_joint">
+        <type>transmission_interface/SimpleTransmission</type>
+        <joint name="meca_axis_6_joint">
+            <hardwareInterface>hardware_interface/EffortJointInterface</hardwareInterface>
+        </joint>
+        <actuator name="meca_axis_6_joint_motor">
+            <hardwareInterface>hardware_interface/EffortJointInterface</hardwareInterface>
+            <mechanicalReduction>1</mechanicalReduction>
+        </actuator>
+    </transmission>
+    <gazebo>
         <plugin name="gazebo_ros_control" filename="libgazebo_ros_control.so">
             <robotNamespace>/</robotNamespace>

Commit message: fixed the joints but controllers still broken on gazebo

File: src/mecademic_description/urdf/meca_500_r3.urdf.xacro (robot description, xacro)
@@ -3,26 +3,9 @@
 <!-- |    This document was autogenerated by xacro from /home/ram/Projects/Project-Interstellar/src/mecademic_description/urdf/meca_500_r3.urdf.xacro | -->
 <!-- |    EDITING THIS FILE BY HAND IS NOT RECOMMENDED                                 | -->
-<!-- =================================================================================== -->
-<!-- =================================================================================== -->
-<!-- |    This document was autogenerated by xacro from /home/ram/Projects/Project-Interstellar/src/mecademic_description/urdf/meca_500_r3.urdf.xacro | -->
-<!-- |    EDITING THIS FILE BY HAND IS NOT RECOMMENDED                                 | -->
-<!-- =================================================================================== -->
-<!-- =================================================================================== -->
-<!-- |    This document was autogenerated by xacro from /home/ram/Projects/Project-Interstellar/src/mecademic_description/urdf/meca_500_r3.urdf.xacro | -->
-<!-- |    EDITING THIS FILE BY HAND IS NOT RECOMMENDED                                 | -->
-<!-- =================================================================================== -->
-<!-- =================================================================================== -->
-<!-- |    This document was autogenerated by xacro from /home/ram/ws_moveit/src/mecademic_description/urdf/meca_500_r3.urdf.xacro | -->
-<!-- |    EDITING THIS FILE BY HAND IS NOT RECOMMENDED                                 | -->
-<!-- =================================================================================== -->
-<!-- =================================================================================== -->
-<!-- |    This document was autogenerated by xacro from /home/ram/ws_moveit/src/mecademic_description/urdf/meca_500_r3.urdf.xacro | -->
-<!-- |    EDITING THIS FILE BY HAND IS NOT RECOMMENDED                                 | -->
-<!-- =================================================================================== -->
 <robot name="meca_500_r3">
-    <link name="world"/>
+    <link name="world" />
     <joint name="fixed" type="fixed">
-        <parent link="world"/>
-        <child link="meca_base_link"/>
+        <parent link="world" />
+        <child link="meca_base_link" />
     </joint>
     <!-- Base link is the center of the robot's bottom plate -->
@@ -522,4 +505,69 @@
     </transmission>
     <gazebo>
+        <plugin filename="libgazebo_ros_control.so" name="gazebo_ros_control">
+            <robotNamespace>/</robotNamespace>
+        </plugin>
+    </gazebo>
+    <transmission name="trans_meca_axis_1_joint">
+        <type>transmission_interface/SimpleTransmission</type>
+        <joint name="meca_axis_1_joint">
+            <hardwareInterface>hardware_interface/PositionJointInterface</hardwareInterface>
+        </joint>
+        <actuator name="meca_axis_1_joint_motor">
+            <hardwareInterface>hardware_interface/PositionJointInterface</hardwareInterface>
+            <mechanicalReduction>1</mechanicalReduction>
+        </actuator>
+    </transmission>
+    <transmission name="trans_meca_axis_2_joint">
+        <type>transmission_interface/SimpleTransmission</type>
+        <joint name="meca_axis_2_joint">
+            <hardwareInterface>hardware_interface/PositionJointInterface</hardwareInterface>
+        </joint>
+        <actuator name="meca_axis_2_joint_motor">
+            <hardwareInterface>hardware_interface/PositionJointInterface</hardwareInterface>
+            <mechanicalReduction>1</mechanicalReduction>
+        </actuator>
+    </transmission>
+    <transmission name="trans_meca_axis_3_joint">
+        <type>transmission_interface/SimpleTransmission</type>
+        <joint name="meca_axis_3_joint">
+            <hardwareInterface>hardware_interface/PositionJointInterface</hardwareInterface>
+        </joint>
+        <actuator name="meca_axis_3_joint_motor">
+            <hardwareInterface>hardware_interface/PositionJointInterface</hardwareInterface>
+            <mechanicalReduction>1</mechanicalReduction>
+        </actuator>
+    </transmission>
+    <transmission name="trans_meca_axis_4_joint">
+        <type>transmission_interface/SimpleTransmission</type>
+        <joint name="meca_axis_4_joint">
+            <hardwareInterface>hardware_interface/PositionJointInterface</hardwareInterface>
+        </joint>
+        <actuator name="meca_axis_4_joint_motor">
+            <hardwareInterface>hardware_interface/PositionJointInterface</hardwareInterface>
+            <mechanicalReduction>1</mechanicalReduction>
+        </actuator>
+    </transmission>
+    <transmission name="trans_meca_axis_5_joint">
+        <type>transmission_interface/SimpleTransmission</type>
+        <joint name="meca_axis_5_joint">
+            <hardwareInterface>hardware_interface/PositionJointInterface</hardwareInterface>
+        </joint>
+        <actuator name="meca_axis_5_joint_motor">
+            <hardwareInterface>hardware_interface/PositionJointInterface</hardwareInterface>
+            <mechanicalReduction>1</mechanicalReduction>
+        </actuator>
+    </transmission>
+    <transmission name="trans_meca_axis_6_joint">
+        <type>transmission_interface/SimpleTransmission</type>
+        <joint name="meca_axis_6_joint">
+            <hardwareInterface>hardware_interface/EffortJointInterface</hardwareInterface>
+        </joint>
+        <actuator name="meca_axis_6_joint_motor">
+            <hardwareInterface>hardware_interface/EffortJointInterface</hardwareInterface>
+            <mechanicalReduction>1</mechanicalReduction>
+        </actuator>
+    </transmission>
+    <gazebo>
         <plugin name="gazebo_ros_control" filename="libgazebo_ros_control.so">
             <robotNamespace>/</robotNamespace>
