Commit message: removed all moveit setup a stuff and rwevert to the old urdf

File: src/mecademic_description/urdf/meca_500_r3.urdf.xacro (robot description, xacro)
@@ -1,1289 +1,149 @@
-<?xml version="1.0" encoding="utf-8"?>
-<!-- =================================================================================== -->
-<!-- |    This document was autogenerated by xacro from /home/ram/Projects/Project-Interstellar/src/mecademic_description/urdf/meca_500_r3.urdf.xacro | -->
-<!-- |    EDITING THIS FILE BY HAND IS NOT RECOMMENDED                                 | -->
-<!-- =================================================================================== -->
-<!-- =================================================================================== -->
-<!-- |    This document was autogenerated by xacro from /home/ram/Projects/Project-Interstellar/src/mecademic_description/urdf/meca_500_r3.urdf.xacro | -->
-<!-- |    EDITING THIS FILE BY HAND IS NOT RECOMMENDED                                 | -->
-<robot name="meca_500_r3">
-    <link name="world" />
-    <joint name="fixed" type="fixed">
-        <parent link="world" />
-        <child link="meca_base_link" />
-    </joint>
-    <!-- Base link is the center of the robot's bottom plate -->
-    <link name="meca_base_link">
-        <visual>
-            <origin rpy="0 0 0" xyz="0 0 0" />
-            <geometry>
-                <mesh filename="package://mecademic_description/meshes/meca_500_r3_base.dae" />
-            </geometry>
-        </visual>
-        <collision>
-            <origin rpy="0 0 0" xyz="0 0 0" />
-            <geometry>
-                <mesh filename="package://mecademic_description/meshes/meca_500_r3_base_collision.stl" />
-            </geometry>
-        </collision>
-        <inertial>
-            <mass value="0.1" />
-            <inertia ixx="0.03" ixy="0.0" ixz="0.0" iyy="0.03" iyz="0.0" izz="0.03" />
-        </inertial>
-    </link>
-    <!-- Joint 1 -->
-    <link name="meca_axis_1_link">
-        <visual>
-            <origin rpy="0 0 0" xyz="0 0 0" />
-            <geometry>
-                <mesh filename="package://mecademic_description/meshes/meca_500_r3_j1.dae" />
-            </geometry>
-        </visual>
-        <collision>
-            <origin rpy="0 0 0" xyz="0 0 0" />
-            <geometry>
-                <mesh filename="package://mecademic_description/meshes/meca_500_r3_j1_collision.stl" />
-            </geometry>
-        </collision>
-        <inertial>
-            <mass value="0.1" />
-            <inertia ixx="0.03" ixy="0.0" ixz="0.0" iyy="0.03" iyz="0.0" izz="0.03" />
-        </inertial>
-    </link>
-    <joint name="meca_axis_1_joint" type="revolute">
-        <origin rpy="0 0 0" xyz="0.012498 0 0.091" />
-        <parent link="meca_base_link" />
-        <child link="meca_axis_1_link" />
-        <axis xyz="0 0 1" />
-        <limit effort="10.0" lower="-3.05433" upper="3.05433" velocity="2.61799" />
-    </joint>
-    <!-- Joint 2 -->
-    <link name="meca_axis_2_link">
-        <visual>
-            <origin rpy="0 0 0" xyz="0 0 0" />
-            <geometry>
-                <mesh filename="package://mecademic_description/meshes/meca_500_r3_j2.dae" />
-            </geometry>
-        </visual>
-        <collision>
-            <origin rpy="0 0 0" xyz="0 0 0" />
-            <geometry>
-                <mesh filename="package://mecademic_description/meshes/meca_500_r3_j2_collision.stl" />
-            </geometry>
-        </collision>
-        <inertial>
-            <mass value="0.1" />
-            <inertia ixx="0.03" ixy="0.0" ixz="0.0" iyy="0.03" iyz="0.0" izz="0.03" />
-        </inertial>
-    </link>
-    <joint name="meca_axis_2_joint" type="revolute">
-        <origin rpy="0 0 0" xyz="0 0 0.044" />
-        <parent link="meca_axis_1_link" />
-        <child link="meca_axis_2_link" />
-        <axis xyz="0 1 0" />
-        <limit effort="10.0" lower="-1.22173048" upper="1.5708" velocity="2.61799" />
-    </joint>
-    <!-- Joint 3 -->
-    <link name="meca_axis_3_link">
-        <visual>
-            <origin rpy="0 0 0" xyz="0 0 0" />
-            <geometry>
-                <mesh filename="package://mecademic_description/meshes/meca_500_r3_j3.dae" />
-            </geometry>
-        </visual>
-        <collision>
-            <origin rpy="0 0 0" xyz="0 0 0" />
-            <geometry>
-                <mesh filename="package://mecademic_description/meshes/meca_500_r3_j3_collision.stl" />
-            </geometry>
-        </collision>
-        <inertial>
-            <mass value="0.1" />
-            <inertia ixx="0.03" ixy="0.0" ixz="0.0" iyy="0.03" iyz="0.0" izz="0.03" />
-        </inertial>
-    </link>
-    <joint name="meca_axis_3_joint" type="revolute">
-        <origin rpy="0 0 0" xyz="0 0 0.135" />
-        <parent link="meca_axis_2_link" />
-        <child link="meca_axis_3_link" />
-        <axis xyz="0 1 0" />
-        <limit effort="10.0" lower="-2.35619" upper="1.22173048" velocity="3.14159" />
-    </joint>
-    <!-- Joint 4 -->
-    <link name="meca_axis_4_link">
-        <visual>
-            <origin rpy="0 0 0" xyz="0 0 0" />
-            <geometry>
-                <mesh filename="package://mecademic_description/meshes/meca_500_r3_j4.dae" />
-            </geometry>
-        </visual>
-        <collision>
-            <origin rpy="0 0 0" xyz="0 0 0" />
-            <geometry>
-                <mesh filename="package://mecademic_description/meshes/meca_500_r3_j4_collision.stl" />
-            </geometry>
-        </collision>
-        <inertial>
-            <mass value="0.1" />
-            <inertia ixx="0.03" ixy="0.0" ixz="0.0" iyy="0.03" iyz="0.0" izz="0.03" />
-        </inertial>
-    </link>
-    <joint name="meca_axis_4_joint" type="revolute">
-        <origin rpy="0 0 0" xyz="0 0 0.038" />
-        <parent link="meca_axis_3_link" />
-        <child link="meca_axis_4_link" />
-        <axis xyz="1 0 0" />
-        <limit effort="10.0" lower="-2.96706" upper="2.96706" velocity="5.23599" />
-    </joint>
-    <!-- Joint 5 -->
-    <link name="meca_axis_5_link">
-        <visual>
-            <origin rpy="0 0 0" xyz="0 0 0" />
-            <geometry>
-                <mesh filename="package://mecademic_description/meshes/meca_500_r3_j5.dae" />
-            </geometry>
-        </visual>
-        <collision>
-            <origin rpy="0 0 0" xyz="0 0 0" />
-            <geometry>
-                <mesh filename="package://mecademic_description/meshes/meca_500_r3_j5_collision.stl" />
-            </geometry>
-        </collision>
-        <inertial>
-            <mass value="0.1" />
-            <inertia ixx="0.03" ixy="0.0" ixz="0.0" iyy="0.03" iyz="0.0" izz="0.03" />
-        </inertial>
-    </link>
-    <joint name="meca_axis_5_joint" type="revolute">
-        <origin rpy="0 0 0" xyz="0.12 0 0" />
-        <parent link="meca_axis_4_link" />
-        <child link="meca_axis_5_link" />
-        <axis xyz="0 1 0" />
-        <limit effort="10.0" lower="-2.00713" upper="2.00713" velocity="5.23599" />
-    </joint>
-    <!-- Joint 6 -->
-    <link name="meca_axis_6_link">
-        <visual>
-            <origin rpy="0 0 0" xyz="0 0 0" />
-            <geometry>
-                <mesh filename="package://mecademic_description/meshes/meca_500_r3_j6.dae" />
-            </geometry>
-        </visual>
-        <collision>
-            <origin rpy="0 0 0" xyz="0 0 0" />
-            <geometry>
-                <mesh filename="package://mecademic_description/meshes/meca_500_r3_j6_collision.stl" />
-            </geometry>
-        </collision>
-        <inertial>
-            <mass value="0.1" />
-            <inertia ixx="0.03" ixy="0.0" ixz="0.0" iyy="0.03" iyz="0.0" izz="0.03" />
-        </inertial>
-    </link>
-    <joint name="meca_axis_6_joint" type="revolute">
-        <origin rpy="0 0 0" xyz="0.07 0 0" />
-        <parent link="meca_axis_5_link" />
-        <child link="meca_axis_6_link" />
-        <axis xyz="1 0 0" />
-        <limit effort="10.0" lower="-3.14159" upper="3.14159" velocity="8.72665" />
-    </joint>
-    <transmission name="trans_meca_axis_1_joint">
-        <type>transmission_interface/SimpleTransmission</type>
-        <joint name="meca_axis_1_joint">
-            <hardwareInterface>hardware_interface/EffortJointInterface</hardwareInterface>
-        </joint>
-        <actuator name="meca_axis_1_joint_motor">
-            <hardwareInterface>hardware_interface/EffortJointInterface</hardwareInterface>
-            <mechanicalReduction>1</mechanicalReduction>
-        </actuator>
-    </transmission>
-    <transmission name="trans_meca_axis_2_joint">
-        <type>transmission_interface/SimpleTransmission</type>
-        <joint name="meca_axis_2_joint">
-            <hardwareInterface>hardware_interface/EffortJointInterface</hardwareInterface>
-        </joint>
-        <actuator name="meca_axis_2_joint_motor">
-            <hardwareInterface>hardware_interface/EffortJointInterface</hardwareInterface>
-            <mechanicalReduction>1</mechanicalReduction>
-        </actuator>
-    </transmission>
-    <transmission name="trans_meca_axis_3_joint">
-        <type>transmission_interface/SimpleTransmission</type>
-        <joint name="meca_axis_3_joint">
-            <hardwareInterface>hardware_interface/EffortJointInterface</hardwareInterface>
-        </joint>
-        <actuator name="meca_axis_3_joint_motor">
-            <hardwareInterface>hardware_interface/EffortJointInterface</hardwareInterface>
-            <mechanicalReduction>1</mechanicalReduction>
-        </actuator>
-    </transmission>
-    <transmission name="trans_meca_axis_4_joint">
-        <type>transmission_interface/SimpleTransmission</type>
-        <joint name="meca_axis_4_joint">
-            <hardwareInterface>hardware_interface/EffortJointInterface</hardwareInterface>
-        </joint>
-        <actuator name="meca_axis_4_joint_motor">
-            <hardwareInterface>hardware_interface/EffortJointInterface</hardwareInterface>
-            <mechanicalReduction>1</mechanicalReduction>
-        </actuator>
-    </transmission>
-    <transmission name="trans_meca_axis_5_joint">
-        <type>transmission_interface/SimpleTransmission</type>
-        <joint name="meca_axis_5_joint">
-            <hardwareInterface>hardware_interface/EffortJointInterface</hardwareInterface>
-        </joint>
-        <actuator name="meca_axis_5_joint_motor">
-            <hardwareInterface>hardware_interface/EffortJointInterface</hardwareInterface>
-            <mechanicalReduction>1</mechanicalReduction>
-        </actuator>
-    </transmission>
-    <transmission name="trans_meca_axis_6_joint">
-        <type>transmission_interface/SimpleTransmission</type>
-        <joint name="meca_axis_6_joint">
-            <hardwareInterface>hardware_interface/EffortJointInterface</hardwareInterface>
-        </joint>
-        <actuator name="meca_axis_6_joint_motor">
-            <hardwareInterface>hardware_interface/EffortJointInterface</hardwareInterface>
-            <mechanicalReduction>1</mechanicalReduction>
-        </actuator>
-    </transmission>
-    <gazebo>
-        <plugin filename="libgazebo_ros_control.so" name="gazebo_ros_control">
-            <robotNamespace>/</robotNamespace>
-        </plugin>
-    </gazebo>
-    <transmission name="trans_meca_axis_1_joint">
-        <type>transmission_interface/SimpleTransmission</type>
-        <joint name="meca_axis_1_joint">
-            <hardwareInterface>hardware_interface/EffortJointInterface</hardwareInterface>
-        </joint>
-        <actuator name="meca_axis_1_joint_motor">
-            <hardwareInterface>hardware_interface/EffortJointInterface</hardwareInterface>
-            <mechanicalReduction>1</mechanicalReduction>
-        </actuator>
-    </transmission>
-    <transmission name="trans_meca_axis_2_joint">
-        <type>transmission_interface/SimpleTransmission</type>
-        <joint name="meca_axis_2_joint">
-            <hardwareInterface>hardware_interface/EffortJointInterface</hardwareInterface>
-        </joint>
-        <actuator name="meca_axis_2_joint_motor">
-            <hardwareInterface>hardware_interface/EffortJointInterface</hardwareInterface>
-            <mechanicalReduction>1</mechanicalReduction>
-        </actuator>
-    </transmission>
-    <transmission name="trans_meca_axis_3_joint">
-        <type>transmission_interface/SimpleTransmission</type>
-        <joint name="meca_axis_3_joint">
-            <hardwareInterface>hardware_interface/EffortJointInterface</hardwareInterface>
-        </joint>
-        <actuator name="meca_axis_3_joint_motor">
-            <hardwareInterface>hardware_interface/EffortJointInterface</hardwareInterface>
-            <mechanicalReduction>1</mechanicalReduction>
-        </actuator>
-    </transmission>
-    <transmission name="trans_meca_axis_4_joint">
-        <type>transmission_interface/SimpleTransmission</type>
-        <joint name="meca_axis_4_joint">
-            <hardwareInterface>hardware_interface/EffortJointInterface</hardwareInterface>
-        </joint>
-        <actuator name="meca_axis_4_joint_motor">
-            <hardwareInterface>hardware_interface/EffortJointInterface</hardwareInterface>
-            <mechanicalReduction>1</mechanicalReduction>
-        </actuator>
-    </transmission>
-    <transmission name="trans_meca_axis_5_joint">
-        <type>transmission_interface/SimpleTransmission</type>
-        <joint name="meca_axis_5_joint">
-            <hardwareInterface>hardware_interface/EffortJointInterface</hardwareInterface>
-        </joint>
-        <actuator name="meca_axis_5_joint_motor">
-            <hardwareInterface>hardware_interface/EffortJointInterface</hardwareInterface>
-            <mechanicalReduction>1</mechanicalReduction>
-        </actuator>
-    </transmission>
-    <transmission name="trans_meca_axis_6_joint">
-        <type>transmission_interface/SimpleTransmission</type>
-        <joint name="meca_axis_6_joint">
-            <hardwareInterface>hardware_interface/EffortJointInterface</hardwareInterface>
-        </joint>
-        <actuator name="meca_axis_6_joint_motor">
-            <hardwareInterface>hardware_interface/EffortJointInterface</hardwareInterface>
-            <mechanicalReduction>1</mechanicalReduction>
-        </actuator>
-    </transmission>
-    <gazebo>
-        <plugin filename="libgazebo_ros_control.so" name="gazebo_ros_control">
-            <robotNamespace>/</robotNamespace>
-        </plugin>
-    </gazebo>
-    <transmission name="trans_meca_axis_1_joint">
-        <type>transmission_interface/SimpleTransmission</type>
-        <joint name="meca_axis_1_joint">
-            <hardwareInterface>hardware_interface/EffortJointInterface</hardwareInterface>
-        </joint>
-        <actuator name="meca_axis_1_joint_motor">
-            <hardwareInterface>hardware_interface/EffortJointInterface</hardwareInterface>
-            <mechanicalReduction>1</mechanicalReduction>
-        </actuator>
-    </transmission>
-    <transmission name="trans_meca_axis_2_joint">
-        <type>transmission_interface/SimpleTransmission</type>
-        <joint name="meca_axis_2_joint">
-            <hardwareInterface>hardware_interface/EffortJointInterface</hardwareInterface>
-        </joint>
-        <actuator name="meca_axis_2_joint_motor">
-            <hardwareInterface>hardware_interface/EffortJointInterface</hardwareInterface>
-            <mechanicalReduction>1</mechanicalReduction>
-        </actuator>
-    </transmission>
-    <transmission name="trans_meca_axis_3_joint">
-        <type>transmission_interface/SimpleTransmission</type>
-        <joint name="meca_axis_3_joint">
-            <hardwareInterface>hardware_interface/EffortJointInterface</hardwareInterface>
-        </joint>
-        <actuator name="meca_axis_3_joint_motor">
-            <hardwareInterface>hardware_interface/EffortJointInterface</hardwareInterface>
-            <mechanicalReduction>1</mechanicalReduction>
-        </actuator>
-    </transmission>
-    <transmission name="trans_meca_axis_4_joint">
-        <type>transmission_interface/SimpleTransmission</type>
-        <joint name="meca_axis_4_joint">
-            <hardwareInterface>hardware_interface/EffortJointInterface</hardwareInterface>
-        </joint>
-        <actuator name="meca_axis_4_joint_motor">
-            <hardwareInterface>hardware_interface/EffortJointInterface</hardwareInterface>
-            <mechanicalReduction>1</mechanicalReduction>
-        </actuator>
-    </transmission>
-    <transmission name="trans_meca_axis_5_joint">
-        <type>transmission_interface/SimpleTransmission</type>
-        <joint name="meca_axis_5_joint">
-            <hardwareInterface>hardware_interface/EffortJointInterface</hardwareInterface>
-        </joint>
-        <actuator name="meca_axis_5_joint_motor">
-            <hardwareInterface>hardware_interface/EffortJointInterface</hardwareInterface>
-            <mechanicalReduction>1</mechanicalReduction>
-        </actuator>
-    </transmission>
-    <transmission name="trans_meca_axis_6_joint">
-        <type>transmission_interface/SimpleTransmission</type>
-        <joint name="meca_axis_6_joint">
-            <hardwareInterface>hardware_interface/EffortJointInterface</hardwareInterface>
-        </joint>
-        <actuator name="meca_axis_6_joint_motor">
-            <hardwareInterface>hardware_interface/EffortJointInterface</hardwareInterface>
-            <mechanicalReduction>1</mechanicalReduction>
-        </actuator>
-    </transmission>
-    <gazebo>
-        <plugin filename="libgazebo_ros_control.so" name="gazebo_ros_control">
-            <robotNamespace>/</robotNamespace>
-        </plugin>
-    </gazebo>
-    <transmission name="trans_meca_axis_1_joint">
-        <type>transmission_interface/SimpleTransmission</type>
-        <joint name="meca_axis_1_joint">
-            <hardwareInterface>hardware_interface/EffortJointInterface</hardwareInterface>
-        </joint>
-        <actuator name="meca_axis_1_joint_motor">
-            <hardwareInterface>hardware_interface/EffortJointInterface</hardwareInterface>
-            <mechanicalReduction>1</mechanicalReduction>
-        </actuator>
-    </transmission>
-    <transmission name="trans_meca_axis_2_joint">
-        <type>transmission_interface/SimpleTransmission</type>
-        <joint name="meca_axis_2_joint">
-            <hardwareInterface>hardware_interface/EffortJointInterface</hardwareInterface>
-        </joint>
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
Commit message: tool and link setup

File: src/mecademic_description/urdf/meca_500_r3.urdf.xacro (robot description, xacro)
@@ -147,3 +147,16 @@
     <limit effort="10.0" velocity="8.72665" lower="-3.14159" upper="3.14159" />
   </joint>
+  <link name="meca_axis_flange" />
+  <joint name="meca_axis_joint_7-flange" type="fixed">
+    <origin xyz="0 0 0" rpy="0 0 0" />
+    <parent link="meca_axis_6_link" />
+    <child link="meca_axis_flange" />
+  </joint>
+  <!-- ROS-Industrial 'tool0' frame: all-zeros tool frame -->
+  <link name="meca_axis_tool0" />
+  <joint name="meca_axis_link_7-tool0" type="fixed">
+    <origin xyz="0 0 0" rpy="${pi} ${-pi/2.0} 0" />
+    <parent link="meca_axis_flange" />
+    <child link="meca_axis_tool0" />
+  </joint>
 </robot>

Commit message: world fix

File: src/mecademic_description/urdf/meca_500_r3.urdf.xacro (robot description, xacro)
@@ -1,4 +1,10 @@
 <robot name="meca_500_r3" xmlns:xacro="http://ros.org/wiki/xacro">
   <!-- Base link is the center of the robot's bottom plate -->
+  <link name="world" />
+  <joint name="world_joint" type="fixed">
+    <parent link="world" />
+    <child link="meca_base_link" />
+    <origin xyz="0.0 0.0 0.0" rpy="0.0 0.0 0.0" />
+  </joint>
   <link name="meca_base_link">
     <visual>
