Commit message: updated setup_assistant

File: src/mecademic_description/urdf/meca_500_r3.urdf.xacro (robot description, xacro)
@@ -1,431 +1,1178 @@
-<robot name="meca_500_r3" xmlns:xacro="http://ros.org/wiki/xacro">
-  <!-- Base link is the center of the robot's bottom plate -->
-  <link name="world" />
-  <joint name="world_joint" type="fixed">
-    <parent link="world" />
-    <child link="meca_base_link" />
-    <origin xyz="0.0 0.0 0.0" rpy="0.0 0.0 0.0" />
-  </joint>
-  <link name="meca_base_link">
-    <visual>
-      <origin xyz="0 0 0" rpy="0 0 0" />
-      <geometry>
-        <mesh filename="package://mecademic_description/meshes/meca_500_r3_base.dae" />
-      </geometry>
-    </visual>
-    <collision>
-      <origin xyz="0 0 0" rpy="0 0 0" />
-      <geometry>
-        <mesh filename="package://mecademic_description/meshes/meca_500_r3_base_collision.stl" />
-      </geometry>
-    </collision>
-  </link>
-  <!-- Joint 1 -->
-  <link name="meca_axis_1_link">
-    <visual>
-      <origin xyz="0 0 0" rpy="0 0 0" />
-      <geometry>
-        <mesh filename="package://mecademic_description/meshes/meca_500_r3_j1.dae" />
-      </geometry>
-    </visual>
-    <collision>
-      <origin xyz="0 0 0" rpy="0 0 0" />
-      <geometry>
-        <mesh filename="package://mecademic_description/meshes/meca_500_r3_j1_collision.stl" />
-      </geometry>
-    </collision>
-  </link>
-  <joint name="meca_axis_1_joint" type="revolute">
-    <origin xyz="0.012498 0 0.091" rpy="0 0 0" />
-    <parent link="meca_base_link" />
-    <child link="meca_axis_1_link" />
-    <axis xyz="0 0 1" />
-    <limit effort="10.0" velocity="2.61799" lower="-3.05433" upper="3.05433" />
-  </joint>
-  <!-- Joint 2 -->
-  <link name="meca_axis_2_link">
-    <visual>
-      <origin xyz="0 0 0" rpy="0 0 0" />
-      <geometry>
-        <mesh filename="package://mecademic_description/meshes/meca_500_r3_j2.dae" />
-      </geometry>
-    </visual>
-    <collision>
-      <origin xyz="0 0 0" rpy="0 0 0" />
-      <geometry>
-        <mesh filename="package://mecademic_description/meshes/meca_500_r3_j2_collision.stl" />
-      </geometry>
-    </collision>
-  </link>
-  <joint name="meca_axis_2_joint" type="revolute">
-    <origin xyz="0 0 0.044" rpy="0 0 0" />
-    <parent link="meca_axis_1_link" />
-    <child link="meca_axis_2_link" />
-    <axis xyz="0 1 0" />
-    <limit effort="10.0" velocity="2.61799" lower="-1.22173048" upper="1.5708" />
-  </joint>
-  <!-- Joint 3 -->
-  <link name="meca_axis_3_link">
-    <visual>
-      <origin xyz="0 0 0" rpy="0 0 0" />
-      <geometry>
-        <mesh filename="package://mecademic_description/meshes/meca_500_r3_j3.dae" />
-      </geometry>
-    </visual>
-    <collision>
-      <origin xyz="0 0 0" rpy="0 0 0" />
-      <geometry>
-        <mesh filename="package://mecademic_description/meshes/meca_500_r3_j3_collision.stl" />
-      </geometry>
-    </collision>
-  </link>
-  <joint name="meca_axis_3_joint" type="revolute">
-    <origin xyz="0 0 0.135" rpy="0 0 0" />
-    <parent link="meca_axis_2_link" />
-    <child link="meca_axis_3_link" />
-    <axis xyz="0 1 0" />
-    <limit effort="10.0" velocity="3.14159" lower="-2.35619" upper="1.22173048" />
-  </joint>
-  <!-- Joint 4 -->
-  <link name="meca_axis_4_link">
-    <visual>
-      <origin xyz="0 0 0" rpy="0 0 0" />
-      <geometry>
-        <mesh filename="package://mecademic_description/meshes/meca_500_r3_j4.dae" />
-      </geometry>
-    </visual>
-    <collision>
-      <origin xyz="0 0 0" rpy="0 0 0" />
-      <geometry>
-        <mesh filename="package://mecademic_description/meshes/meca_500_r3_j4_collision.stl" />
-      </geometry>
-    </collision>
-  </link>
-  <joint name="meca_axis_4_joint" type="revolute">
-    <origin xyz="0 0 0.038" rpy="0 0 0" />
-    <parent link="meca_axis_3_link" />
-    <child link="meca_axis_4_link" />
-    <axis xyz="1 0 0" />
-    <limit effort="10.0" velocity="5.23599" lower="-2.96706" upper="2.96706" />
-  </joint>
-  <!-- Joint 5 -->
-  <link name="meca_axis_5_link">
-    <visual>
-      <origin xyz="0 0 0" rpy="0 0 0" />
-      <geometry>
-        <mesh filename="package://mecademic_description/meshes/meca_500_r3_j5.dae" />
-      </geometry>
-    </visual>
-    <collision>
-      <origin xyz="0 0 0" rpy="0 0 0" />
-      <geometry>
-        <mesh filename="package://mecademic_description/meshes/meca_500_r3_j5_collision.stl" />
-      </geometry>
-    </collision>
-  </link>
-  <joint name="meca_axis_5_joint" type="revolute">
-    <origin xyz="0.12 0 0" rpy="0 0 0" />
-    <parent link="meca_axis_4_link" />
-    <child link="meca_axis_5_link" />
-    <axis xyz="0 1 0" />
-    <limit effort="10.0" velocity="5.23599" lower="-2.00713" upper="2.00713" />
-  </joint>
-  <!-- Joint 6 -->
-  <link name="meca_axis_6_link">
-    <visual>
-      <origin xyz="0 0 0" rpy="0 0 0" />
-      <geometry>
-        <mesh filename="package://mecademic_description/meshes/meca_500_r3_j6.dae" />
-      </geometry>
-    </visual>
-    <collision>
-      <origin xyz="0 0 0" rpy="0 0 0" />
-      <geometry>
-        <mesh filename="package://mecademic_description/meshes/meca_500_r3_j6_collision.stl" />
-      </geometry>
-    </collision>
-  </link>
-  <joint name="meca_axis_6_joint" type="revolute">
-    <origin xyz="0.07 0 0" rpy="0 0 0" />
-    <parent link="meca_axis_5_link" />
-    <child link="meca_axis_6_link" />
-    <axis xyz="1 0 0" />
-    <limit effort="10.0" velocity="8.72665" lower="-3.14159" upper="3.14159" />
-  </joint>
-  <link name="meca_axis_flange" />
-  <joint name="meca_axis_joint_7-flange" type="fixed">
-    <origin xyz="0 0 0" rpy="0 0 0" />
-    <parent link="meca_axis_6_link" />
-    <child link="meca_axis_flange" />
-  </joint>
-  <!-- ROS-Industrial 'tool0' frame: all-zeros tool frame -->
-  <link name="meca_axis_tool0" />
-  <joint name="meca_axis_link_7-tool0" type="fixed">
-    <origin xyz="0 0 0" rpy="${pi} ${-pi/2.0} 0" />
-    <parent link="meca_axis_flange" />
-    <child link="meca_axis_tool0" />
-  </joint>
-  <!-- End Effector -->
-  <joint name="meca_axis_link_end_effector" type="fixed">
-    <origin xyz="0 0 0" rpy="${pi} ${pi} 0" />
-    <parent link="meca_axis_tool0" />
-    <child link="robotiq_85_base_link" />
-  </joint>
-  <link name="robotiq_85_base_link">
-    <inertial>
-      <origin xyz="0.00021987 -2.3546E-10 0.030163" rpy="0 0 0" />
-      <mass value="0.30915" />
-      <inertia ixx="0.00028972" ixy="-5.7879E-10" ixz="-1.8543E-06" iyy="0.00030737" iyz="1.682E-12" izz="0.00019914" />
-    </inertial>
-    <visual>
-      <origin xyz="0 0 0" rpy="0 0 0" />
-      <geometry>
-        <mesh filename="package://mecademic_description/meshes/robotiq_85_base_link_fine.STL" />
-      </geometry>
-      <material name="">
-        <color rgba="0.1 0.1 0.1 1" />
-      </material>
-    </visual>
-    <collision>
-      <origin xyz="0 0 0" rpy="0 0 0" />
-      <geometry>
-        <mesh filename="package://mecademic_description/meshes/robotiq_85_base_link_coarse.STL" />
-      </geometry>
-    </collision>
-  </link>
-  <link name="left_outer_knuckle">
-    <inertial>
-      <origin xyz="0.0178331863169983 3.68915177224286E-11 0.0021442477325704" rpy="0 0 0" />
-      <mass value="0.00684838849434396" />
-      <inertia ixx="2.66832029033166E-07" ixy="1.66142314639824E-15" ixz="1.45945633322873E-07" iyy="1.3889233257419E-06" iyz="2.82951161241588E-15" izz="1.26603336914415E-06" />
-    </inertial>
-    <visual>
-      <origin xyz="0 0 0" rpy="0 0 0" />
-      <geometry>
-        <mesh filename="package://mecademic_description/meshes/outer_knuckle_fine.STL" />
-      </geometry>
-      <material name="">
-        <color rgba="0.1 0.1 0.1 1" />
-      </material>
-    </visual>
-    <collision>
-      <origin xyz="0 0 0" rpy="0 0 0" />
-      <geometry>
-        <mesh filename="package://mecademic_description/meshes/outer_knuckle_coarse.STL" />
-      </geometry>
-    </collision>
-  </link>
-  <joint name="finger_joint" type="revolute">
-    <origin xyz="0.0306011444260539 0 0.0627920162695395" rpy="0 0 0" />
-    <parent link="robotiq_85_base_link" />
-    <child link="left_outer_knuckle" />
-    <axis xyz="0 -1 0" />
-    <limit lower="0" upper="0.725" velocity="2.0" effort="1000" />
-  </joint>
-  <link name="left_outer_finger">
-    <inertial>
-      <origin xyz="0.00131451599174296 2.88942057994543E-15 0.0215404163180413" rpy="0 0 0" />
-      <mass value="0.0273093985570947" />
-      <inertia ixx="8.51629628283022E-06" ixy="2.58174336207405E-19" ixz="3.83829504344079E-07" iyy="6.9133328065108E-06" iyz="-7.58589926143789E-19" izz="2.25006832221981E-06" />
-    </inertial>
-    <visual>
-      <origin xyz="0 0 0" rpy="0 0 0" />
-      <geometry>
-        <mesh filename="package://mecademic_description/meshes/outer_finger_fine.STL" />
-      </geometry>
-      <material name="">
-        <color rgba="0.1 0.1 0.1 1" />
-      </material>
-    </visual>
-    <collision>
-      <origin xyz="0 0 0" rpy="0 0 0" />
-      <geometry>
-        <mesh filename="package://mecademic_description/meshes/outer_finger_coarse.STL" />
-      </geometry>
-    </collision>
-  </link>
-  <joint name="left_outer_finger_joint" type="fixed">
-    <origin xyz="0.0316910442266543 0 -0.00193396375724605" rpy="0 0 0" />
-    <parent link="left_outer_knuckle" />
-    <child link="left_outer_finger" />
-    <axis xyz="0 -1 0" />
-  </joint>
-  <link name="left_inner_knuckle">
-    <inertial>
-      <origin xyz="0.017097546626628 -3.93808524389535E-10 0.0224918438201868" rpy="0 0 0" />
-      <mass value="0.0110930853895903" />
-      <inertia ixx="4.23392770691541E-06" ixy="5.748978936968E-15" ixz="1.78855677119788E-06" iyy="3.96548790524392E-06" iyz="1.05464666369669E-14" izz="3.24068002883007E-06" />
-    </inertial>
-    <visual>
-      <origin xyz="0 0 0" rpy="0 0 0" />
-      <geometry>
-        <mesh filename="package://mecademic_description/meshes/inner_knuckle_fine.STL" />
-      </geometry>
-      <material name="">
-        <color rgba="0.1 0.1 0.1 1" />
-      </material>
-    </visual>
-    <collision>
-      <origin xyz="0 0 0" rpy="0 0 0" />
-      <geometry>
-        <mesh filename="package://mecademic_description/meshes/inner_knuckle_coarse.STL" />
-      </geometry>
-    </collision>
-  </link>
-  <joint name="left_inner_knuckle_joint" type="revolute">
-    <origin xyz="0.0127000000001501 0 0.0693074999999639" rpy="0 0 0" />
-    <parent link="robotiq_85_base_link" />
-    <child link="left_inner_knuckle" />
-    <axis xyz="0 -1 0" />
-    <limit lower="0" upper="0.8757" velocity="2.0" effort="1000" />
-    <mimic joint="finger_joint" multiplier="1" offset="0" />
-  </joint>
-  <link name="left_inner_finger">
-    <inertial>
-      <origin xyz="0.0060275613594574 -6.29183141465421E-15 0.00669925693133241" rpy="0 0 0" />
-      <mass value="0.00724255346165745" />
-      <inertia ixx="1.47824274053603E-06" ixy="-3.94884463570303E-19" ixz="-3.45268847648622E-07" iyy="1.70064480838395E-06" iyz="3.5059838910097E-19" izz="4.77151336838364E-07" />
-    </inertial>
-    <visual>
-      <origin xyz="0 0 0" rpy="0 0 0" />
-      <geometry>
-        <mesh filename="package://mecademic_description/meshes/inner_finger_fine.STL" />
-      </geometry>
-      <material name="">
-        <color rgba="0.1 0.1 0.1 1" />
-      </material>
-    </visual>
-    <collision>
-      <origin xyz="0 0 0" rpy="0 0 0" />
-      <geometry>
-        <mesh filename="package://mecademic_description/meshes/inner_finger_coarse.STL" />
-      </geometry>
-    </collision>
-  </link>
-  <joint name="left_inner_finger_joint" type="revolute">
-    <origin xyz="0.034585310861294 0 0.0454970193817975" rpy="0 0 0" />
-    <parent link="left_inner_knuckle" />
-    <child link="left_inner_finger" />
-    <axis xyz="0 -1 0" />
-    <limit lower="0" upper="0.8757" velocity="2.0" effort="1000" />
-    <mimic joint="finger_joint" multiplier="-1" offset="0" />
-  </joint>
-  <link name="right_inner_knuckle">
-    <inertial>
-      <origin xyz="0.0168606186773776 3.93808471820465E-10 0.0226699950793434" rpy="0 0 0" />
-      <mass value="0.0110930853895903" />
-      <inertia ixx="4.27134775939882E-06" ixy="-8.53568456728898E-15" ixz="1.77774229944246E-06" iyy="3.96548790524392E-06" iyz="-8.45108024914164E-15" izz="3.20325997634666E-06" />
-    </inertial>
-    <visual>
-      <origin xyz="0 0 0" rpy="0 0 0" />
-      <geometry>
-        <mesh filename="package://mecademic_description/meshes/inner_knuckle_fine.STL" />
-      </geometry>
-      <material name="">
-        <color rgba="0.1 0.1 0.1 1" />
-      </material>
-    </visual>
-    <collision>
-      <origin xyz="0 0 0" rpy="0 0 0" />
-      <geometry>
-        <mesh filename="package://mecademic_description/meshes/inner_knuckle_coarse.STL" />
-      </geometry>
-    </collision>
-  </link>
-  <joint name="right_inner_knuckle_joint" type="revolute">
-    <origin xyz="-0.0126999999998499 0 0.0693075000000361" rpy="0 0 3.14159265358979" />
-    <parent link="robotiq_85_base_link" />
-    <child link="right_inner_knuckle" />
-    <axis xyz="0 1 0" />
-    <limit lower="0" upper="0.8757" velocity="2.0" effort="1000" />
-    <mimic joint="finger_joint" multiplier="-1" offset="0" />
-  </joint>
-  <link name="right_inner_finger">
-    <inertial>
-      <origin xyz="0.00602756228812038 -6.47284509480176E-15 0.00669925609578108" rpy="0 0 0" />
-      <mass value="0.00724255346165744" />
-      <inertia ixx="1.47824283625957E-06" ixy="-3.95952064019123E-19" ixz="-3.45268708875543E-07" iyy="1.70064480838394E-06" iyz="3.55286507960029E-19" izz="4.77151241114822E-07" />
-    </inertial>
-    <visual>
-      <origin xyz="0 0 0" rpy="0 0 0" />
-      <geometry>
-        <mesh filename="package://mecademic_description/meshes/inner_finger_fine.STL" />
-      </geometry>
-      <material name="">
-        <color rgba="0.1 0.1 0.1 1" />
-      </material>
-    </visual>
-    <collision>
-      <origin xyz="0 0 0" rpy="0 0 0" />
-      <geometry>
-        <mesh filename="package://mecademic_description/meshes/inner_finger_coarse.STL" />
-      </geometry>
-    </collision>
-  </link>
-  <joint name="right_inner_finger_joint" type="revolute">
-    <origin xyz="0.0341060475457406 0 0.0458573878541688" rpy="0 0 0" />
-    <parent link="right_inner_knuckle" />
-    <child link="right_inner_finger" />
-    <axis xyz="0 1 0" />
-    <limit lower="0" upper="0.8757" velocity="2.0" effort="1000" />
-    <mimic joint="finger_joint" multiplier="1" offset="0" />
-  </joint>
-  <link name="right_outer_knuckle">
-    <inertial>
-      <origin xyz="0.0178097074051638 3.60493211424024E-11 0.00233123458346721" rpy="0 0 0" />
-      <mass value="0.00684838849401352" />
-      <inertia ixx="2.70004361573169E-07" ixy="1.59579467624491E-15" ixz="1.56396493788199E-07" iyy="1.38892332558312E-06" iyz="2.82357800318817E-15" izz="1.26286103637978E-06" />
-    </inertial>
-    <visual>
-      <origin xyz="0 0 0" rpy="0 0 0" />
-      <geometry>
-        <mesh filename="package://mecademic_description/meshes/outer_knuckle_fine.STL" />
-      </geometry>
-      <material name="">
-        <color rgba="0.1 0.1 0.1 1" />
-      </material>
-    </visual>
-    <collision>
-      <origin xyz="0 0 0" rpy="0 0 0" />
-      <geometry>
-        <mesh filename="package://mecademic_description/meshes/outer_knuckle_coarse.STL" />
-      </geometry>
-    </collision>
-  </link>
-  <joint name="right_outer_knuckle_joint" type="revolute">
-    <origin xyz="-0.0306011444258893 0 0.0627920162695395" rpy="0 0 3.14159265358979" />
-    <parent link="robotiq_85_base_link" />
-    <child link="right_outer_knuckle" />
-    <axis xyz="0 1 0" />
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