Commit message: ros controller issue fixed. but the end effector is not working correctly

File: src/mecademic_description/urdf/meca_500_r3.urdf.xacro (robot description, xacro)
@@ -1,3 +1,3 @@
-<?xml version="1.0" encoding="utf-8" ?>
+<?xml version="1.0" encoding="utf-8"?>
 <!-- =================================================================================== -->
 <!-- |    This document was autogenerated by xacro from /home/ram/Projects/Project-Interstellar/src/mecademic_description/urdf/meca_500_r3.urdf.xacro | -->
@@ -25,7 +25,7 @@
             </geometry>
         </collision>
-<inertial>
+        <inertial>
             <mass value="0.1" />
-            <inertia ixx="0.03" iyy="0.03" izz="0.03" ixy="0.0" ixz="0.0" iyz="0.0" />
+            <inertia ixx="0.03" ixy="0.0" ixz="0.0" iyy="0.03" iyz="0.0" izz="0.03" />
         </inertial>
     </link>
@@ -44,7 +44,7 @@
             </geometry>
         </collision>
-<inertial>
+        <inertial>
             <mass value="0.1" />
-            <inertia ixx="0.03" iyy="0.03" izz="0.03" ixy="0.0" ixz="0.0" iyz="0.0" />
+            <inertia ixx="0.03" ixy="0.0" ixz="0.0" iyy="0.03" iyz="0.0" izz="0.03" />
         </inertial>
     </link>
@@ -70,7 +70,7 @@
             </geometry>
         </collision>
-<inertial>
+        <inertial>
             <mass value="0.1" />
-            <inertia ixx="0.03" iyy="0.03" izz="0.03" ixy="0.0" ixz="0.0" iyz="0.0" />
+            <inertia ixx="0.03" ixy="0.0" ixz="0.0" iyy="0.03" iyz="0.0" izz="0.03" />
         </inertial>
     </link>
@@ -96,7 +96,7 @@
             </geometry>
         </collision>
-<inertial>
+        <inertial>
             <mass value="0.1" />
-            <inertia ixx="0.03" iyy="0.03" izz="0.03" ixy="0.0" ixz="0.0" iyz="0.0" />
+            <inertia ixx="0.03" ixy="0.0" ixz="0.0" iyy="0.03" iyz="0.0" izz="0.03" />
         </inertial>
     </link>
@@ -122,7 +122,7 @@
             </geometry>
         </collision>
-<inertial>
+        <inertial>
             <mass value="0.1" />
-            <inertia ixx="0.03" iyy="0.03" izz="0.03" ixy="0.0" ixz="0.0" iyz="0.0" />
+            <inertia ixx="0.03" ixy="0.0" ixz="0.0" iyy="0.03" iyz="0.0" izz="0.03" />
         </inertial>
     </link>
@@ -148,7 +148,7 @@
             </geometry>
         </collision>
-<inertial>
+        <inertial>
             <mass value="0.1" />
-            <inertia ixx="0.03" iyy="0.03" izz="0.03" ixy="0.0" ixz="0.0" iyz="0.0" />
+            <inertia ixx="0.03" ixy="0.0" ixz="0.0" iyy="0.03" iyz="0.0" izz="0.03" />
         </inertial>
     </link>
@@ -174,7 +174,7 @@
             </geometry>
         </collision>
-<inertial>
+        <inertial>
             <mass value="0.1" />
-            <inertia ixx="0.03" iyy="0.03" izz="0.03" ixy="0.0" ixz="0.0" iyz="0.0" />
+            <inertia ixx="0.03" ixy="0.0" ixz="0.0" iyy="0.03" iyz="0.0" izz="0.03" />
         </inertial>
     </link>
@@ -206,5 +206,5 @@
     </joint>
     <link name="robotiq_85_base_link">
-<inertial>
+        <inertial>
             <origin rpy="0 0 0" xyz="0.00021987 -2.3546E-10 0.030163" />
             <mass value="0.30915" />
@@ -228,5 +228,5 @@
     </link>
     <link name="left_outer_knuckle">
-<inertial>
+        <inertial>
             <origin rpy="0 0 0" xyz="0.0178331863169983 3.68915177224286E-11 0.0021442477325704" />
             <mass value="0.00684838849434396" />
@@ -257,5 +257,5 @@
     </joint>
     <link name="left_outer_finger">
-<inertial>
+        <inertial>
             <origin rpy="0 0 0" xyz="0.00131451599174296 2.88942057994543E-15 0.0215404163180413" />
             <mass value="0.0273093985570947" />
@@ -285,5 +285,5 @@
     </joint>
     <link name="left_inner_knuckle">
-<inertial>
+        <inertial>
             <origin rpy="0 0 0" xyz="0.017097546626628 -3.93808524389535E-10 0.0224918438201868" />
             <mass value="0.0110930853895903" />
@@ -315,5 +315,5 @@
     </joint>
     <link name="left_inner_finger">
-<inertial>
+        <inertial>
             <origin rpy="0 0 0" xyz="0.0060275613594574 -6.29183141465421E-15 0.00669925693133241" />
             <mass value="0.00724255346165745" />
@@ -345,5 +345,5 @@
     </joint>
     <link name="right_inner_knuckle">
-<inertial>
+        <inertial>
             <origin rpy="0 0 0" xyz="0.0168606186773776 3.93808471820465E-10 0.0226699950793434" />
             <mass value="0.0110930853895903" />
@@ -375,5 +375,5 @@
     </joint>
     <link name="right_inner_finger">
-<inertial>
+        <inertial>
             <origin rpy="0 0 0" xyz="0.00602756228812038 -6.47284509480176E-15 0.00669925609578108" />
             <mass value="0.00724255346165744" />
@@ -405,5 +405,5 @@
     </joint>
     <link name="right_outer_knuckle">
-<inertial>
+        <inertial>
             <origin rpy="0 0 0" xyz="0.0178097074051638 3.60493211424024E-11 0.00233123458346721" />
             <mass value="0.00684838849401352" />
@@ -435,5 +435,5 @@
     </joint>
     <link name="right_outer_finger">
-<inertial>
+        <inertial>
             <origin rpy="0 0 0" xyz="0.00108844269639009 -2.611488350845E-15 0.0215530225245502" />
             <mass value="0.0273093985570947" />
@@ -462,5 +462,5 @@
         <axis xyz="0 1 0" />
     </joint>
-<transmission name="trans_meca_axis_1_joint">
+    <transmission name="trans_meca_axis_1_joint">
         <type>transmission_interface/SimpleTransmission</type>
         <joint name="meca_axis_1_joint">
@@ -519,4 +519,129 @@
         <actuator name="meca_axis_6_joint_motor">
             <hardwareInterface>hardware_interface/EffortJointInterface</hardwareInterface>
+            <mechanicalReduction>1</mechanicalReduction>
+        </actuator>
+    </transmission>
+    <transmission name="trans_finger_joint">
+        <type>transmission_interface/SimpleTransmission</type>
+        <joint name="finger_joint">
+            <hardwareInterface>hardware_interface/EffortJointInterface</hardwareInterface>
+        </joint>
+        <actuator name="finger_joint_motor">
+            <hardwareInterface>hardware_interface/EffortJointInterface</hardwareInterface>
+            <mechanicalReduction>1</mechanicalReduction>
+        </actuator>
+    </transmission>
+    <transmission name="trans_left_inner_knuckle_joint">
+        <type>transmission_interface/SimpleTransmission</type>
+        <joint name="left_inner_knuckle_joint">
+            <hardwareInterface>hardware_interface/EffortJointInterface</hardwareInterface>
+        </joint>
+        <actuator name="left_inner_knuckle_joint_motor">
+            <hardwareInterface>hardware_interface/EffortJointInterface</hardwareInterface>
+            <mechanicalReduction>1</mechanicalReduction>
+        </actuator>
+    </transmission>
+    <transmission name="trans_left_inner_finger_joint">
+        <type>transmission_interface/SimpleTransmission</type>
+        <joint name="left_inner_finger_joint">
+            <hardwareInterface>hardware_interface/EffortJointInterface</hardwareInterface>
+        </joint>
+        <actuator name="left_inner_finger_joint_motor">
+            <hardwareInterface>hardware_interface/EffortJointInterface</hardwareInterface>
+            <mechanicalReduction>1</mechanicalReduction>
+        </actuator>
+    </transmission>
+    <transmission name="trans_right_inner_knuckle_joint">
+        <type>transmission_interface/SimpleTransmission</type>
+        <joint name="right_inner_knuckle_joint">
+            <hardwareInterface>hardware_interface/EffortJointInterface</hardwareInterface>
+        </joint>
+        <actuator name="right_inner_knuckle_joint_motor">
+            <hardwareInterface>hardware_interface/EffortJointInterface</hardwareInterface>
+            <mechanicalReduction>1</mechanicalReduction>
+        </actuator>
+    </transmission>
+    <transmission name="trans_right_inner_finger_joint">
+        <type>transmission_interface/SimpleTransmission</type>
+        <joint name="right_inner_finger_joint">
+            <hardwareInterface>hardware_interface/EffortJointInterface</hardwareInterface>
+        </joint>
+        <actuator name="right_inner_finger_joint_motor">
+            <hardwareInterface>hardware_interface/EffortJointInterface</hardwareInterface>
+            <mechanicalReduction>1</mechanicalReduction>
+        </actuator>
+    </transmission>
+    <transmission name="trans_right_outer_knuckle_joint">
+        <type>transmission_interface/SimpleTransmission</type>
+        <joint name="right_outer_knuckle_joint">
+            <hardwareInterface>hardware_interface/EffortJointInterface</hardwareInterface>
+        </joint>
+        <actuator name="right_outer_knuckle_joint_motor">
+            <hardwareInterface>hardware_interface/EffortJointInterface</hardwareInterface>
+            <mechanicalReduction>1</mechanicalReduction>
+        </actuator>
+    </transmission>
+    <gazebo>
+        <plugin filename="libgazebo_ros_control.so" name="gazebo_ros_control">
+            <robotNamespace>/</robotNamespace>
+        </plugin>
+    </gazebo>
+    <transmission name="trans_meca_axis_1_joint">
+        <type>transmission_interface/SimpleTransmission</type>
+        <joint name="meca_axis_1_joint">
+            <hardwareInterface>hardware_interface/PositionJointInterface</hardwareInterface>
+        </joint>
+        <actuator name="meca_axis_1_joint_motor">
+            <hardwareInterface>hardware_interface/PositionJointInterface</hardwareInterface>
+            <mechanicalReduction>1</mechanicalReduction>
+        </actuator>
+    </transmission>
+    <transmission name="trans_meca_axis_2_joint">
+        <type>transmission_interface/SimpleTransmission</type>
+        <joint name="meca_axis_2_joint">
+            <hardwareInterface>hardware_interface/PositionJointInterface</hardwareInterface>
+        </joint>
+        <actuator name="meca_axis_2_joint_motor">
+            <hardwareInterface>hardware_interface/PositionJointInterface</hardwareInterface>
+            <mechanicalReduction>1</mechanicalReduction>
+        </actuator>
+    </transmission>
+    <transmission name="trans_meca_axis_3_joint">
+        <type>transmission_interface/SimpleTransmission</type>
+        <joint name="meca_axis_3_joint">
+            <hardwareInterface>hardware_interface/PositionJointInterface</hardwareInterface>
+        </joint>
+        <actuator name="meca_axis_3_joint_motor">
+            <hardwareInterface>hardware_interface/PositionJointInterface</hardwareInterface>
+            <mechanicalReduction>1</mechanicalReduction>
+        </actuator>
+    </transmission>
+    <transmission name="trans_meca_axis_4_joint">
+        <type>transmission_interface/SimpleTransmission</type>
+        <joint name="meca_axis_4_joint">
+            <hardwareInterface>hardware_interface/PositionJointInterface</hardwareInterface>
+        </joint>
+        <actuator name="meca_axis_4_joint_motor">
+            <hardwareInterface>hardware_interface/PositionJointInterface</hardwareInterface>
+            <mechanicalReduction>1</mechanicalReduction>
+        </actuator>
+    </transmission>
+    <transmission name="trans_meca_axis_5_joint">
+        <type>transmission_interface/SimpleTransmission</type>
+        <joint name="meca_axis_5_joint">
+            <hardwareInterface>hardware_interface/PositionJointInterface</hardwareInterface>
+        </joint>
+        <actuator name="meca_axis_5_joint_motor">
+            <hardwareInterface>hardware_interface/PositionJointInterface</hardwareInterface>
+            <mechanicalReduction>1</mechanicalReduction>
+        </actuator>
+    </transmission>
+    <transmission name="trans_meca_axis_6_joint">
+        <type>transmission_interface/SimpleTransmission</type>
+        <joint name="meca_axis_6_joint">
+            <hardwareInterface>hardware_interface/PositionJointInterface</hardwareInterface>
+        </joint>
+        <actuator name="meca_axis_6_joint_motor">
+            <hardwareInterface>hardware_interface/PositionJointInterface</hardwareInterface>
             <mechanicalReduction>1</mechanicalReduction>
         </actuator>
@@ -588,591 +713,2 @@
     </gazebo>
 </robot>
-<?xml version="1.0" encoding="utf-8" ?>
-<!-- =================================================================================== -->
-<!-- |    This document was autogenerated by xacro from /home/ram/Projects/Project-Interstellar/src/mecademic_description/urdf/meca_500_r3.urdf.xacro | -->
-<!-- |    EDITING THIS FILE BY HAND IS NOT RECOMMENDED                                 | -->
-<!-- =================================================================================== -->
-<robot name="meca_500_r3">
-    <!-- Base link is the center of the robot's bottom plate -->
-    <link name="world" />
-    <joint name="world_joint" type="fixed">
-        <parent link="world" />
-        <child link="meca_base_link" />
-        <origin rpy="0.0 0.0 0.0" xyz="0.0 0.0 0.0" />
-    </joint>
-    <link name="meca_base_link">
-        <visual>
-            <origin rpy="0 0 0" xyz="0 0 0" />
-            <geometry>
-                <mesh filename="package://mecademic_description/meshes/meca_500_r3_base.dae" />
-            </geometry>
-        </visual>
-        <collision>
-            <origin rpy="0 0 0" xyz="0 0 0" />
-            <geometry>
-                <mesh filename="package://mecademic_description/meshes/meca_500_r3_base_collision.stl" />
-            </geometry>
-        </collision>
-<inertial>
-            <mass value="0.1" />
-            <inertia ixx="0.03" iyy="0.03" izz="0.03" ixy="0.0" ixz="0.0" iyz="0.0" />
-        </inertial>
-    </link>
-    <!-- Joint 1 -->
-    <link name="meca_axis_1_link">
-        <visual>
-            <origin rpy="0 0 0" xyz="0 0 0" />
-            <geometry>
-                <mesh filename="package://mecademic_description/meshes/meca_500_r3_j1.dae" />
-            </geometry>
-        </visual>
-        <collision>
-            <origin rpy="0 0 0" xyz="0 0 0" />
-            <geometry>
-                <mesh filename="package://mecademic_description/meshes/meca_500_r3_j1_collision.stl" />
-            </geometry>
-        </collision>
-<inertial>
-            <mass value="0.1" />
-            <inertia ixx="0.03" iyy="0.03" izz="0.03" ixy="0.0" ixz="0.0" iyz="0.0" />
-        </inertial>
-    </link>
-    <joint name="meca_axis_1_joint" type="revolute">
-        <origin rpy="0 0 0" xyz="0.012498 0 0.091" />
-        <parent link="meca_base_link" />
-        <child link="meca_axis_1_link" />
-        <axis xyz="0 0 1" />
-        <limit effort="10.0" lower="-3.05433" upper="3.05433" velocity="2.61799" />
-    </joint>
-    <!-- Joint 2 -->
-    <link name="meca_axis_2_link">
-        <visual>
-            <origin rpy="0 0 0" xyz="0 0 0" />
-            <geometry>
-                <mesh filename="package://mecademic_description/meshes/meca_500_r3_j2.dae" />
-            </geometry>
-        </visual>
-        <collision>
-            <origin rpy="0 0 0" xyz="0 0 0" />
-            <geometry>
-                <mesh filename="package://mecademic_description/meshes/meca_500_r3_j2_collision.stl" />
-            </geometry>
-        </collision>
-<inertial>
-            <mass value="0.1" />
-            <inertia ixx="0.03" iyy="0.03" izz="0.03" ixy="0.0" ixz="0.0" iyz="0.0" />
-        </inertial>
-    </link>
-    <joint name="meca_axis_2_joint" type="revolute">
-        <origin rpy="0 0 0" xyz="0 0 0.044" />
-        <parent link="meca_axis_1_link" />
-        <child link="meca_axis_2_link" />
-        <axis xyz="0 1 0" />
-        <limit effort="10.0" lower="-1.22173048" upper="1.5708" velocity="2.61799" />
-    </joint>
-    <!-- Joint 3 -->
-    <link name="meca_axis_3_link">
-        <visual>
-            <origin rpy="0 0 0" xyz="0 0 0" />
-            <geometry>
-                <mesh filename="package://mecademic_description/meshes/meca_500_r3_j3.dae" />
-            </geometry>
-        </visual>
-        <collision>
-            <origin rpy="0 0 0" xyz="0 0 0" />
-            <geometry>
-                <mesh filename="package://mecademic_description/meshes/meca_500_r3_j3_collision.stl" />
-            </geometry>
-        </collision>
-<inertial>
-            <mass value="0.1" />
-            <inertia ixx="0.03" iyy="0.03" izz="0.03" ixy="0.0" ixz="0.0" iyz="0.0" />
-        </inertial>
-    </link>
-    <joint name="meca_axis_3_joint" type="revolute">
-        <origin rpy="0 0 0" xyz="0 0 0.135" />
-        <parent link="meca_axis_2_link" />
-        <child link="meca_axis_3_link" />
-        <axis xyz="0 1 0" />
-        <limit effort="10.0" lower="-2.35619" upper="1.22173048" velocity="3.14159" />
-    </joint>
-    <!-- Joint 4 -->
-    <link name="meca_axis_4_link">
-        <visual>
-            <origin rpy="0 0 0" xyz="0 0 0" />
-            <geometry>
-                <mesh filename="package://mecademic_description/meshes/meca_500_r3_j4.dae" />
-            </geometry>
-        </visual>
-        <collision>
-            <origin rpy="0 0 0" xyz="0 0 0" />
-            <geometry>
-                <mesh filename="package://mecademic_description/meshes/meca_500_r3_j4_collision.stl" />
-            </geometry>
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