Commit message: collision fix

File: src/mecademic_description/urdf/meca_500_r3.urdf.xacro (robot description, xacro)
@@ -212,10 +212,10 @@
         </visual>
         <collision>
-            <origin rpy="0 1.57079632679 1.57079632679" xyz="0 0 0.04" />
-            <geometry>
-                <cylinder length="0.1" radius="0.07" />
-            </geometry>
-        </collision>
-        <collision>
+            <origin rpy="0 1.57079632679 1.57079632679" xyz="0 0 0.03" />
+            <geometry>
+                <box size="0.07 0.04 0.2" />
+            </geometry>
+        </collision>
+        <!-- <collision>
             <origin rpy="0 0 0" xyz="0 -0.05 0.04" />
             <geometry>
@@ -228,6 +228,6 @@
                 <sphere radius="0.07" />
             </geometry>
-        </collision>
-        <collision>
+        </collision> -->
+        <!-- <collision>
             <origin rpy="0 1.57079632679 1.57079632679" xyz="0 0 0.1" />
             <geometry>
@@ -246,5 +246,5 @@
                 <sphere radius="0.05" />
             </geometry>
-        </collision>
+        </collision> -->
         <inertial>
             <mass value="0.1" />
@@ -262,4 +262,10 @@
             <inertia ixx="0.03" iyy="0.03" izz="0.03" ixy="0.0" ixz="0.0" iyz="0.0" />
         </inertial>
+        <collision>
+            <origin rpy="0 0 0" xyz="0 0 0" />
+            <geometry>
+                <mesh filename="package://mecademic_description/meshes/finger.dae" />
+            </geometry>
+        </collision>
     </link>
     <link name="meca_rightfinger">
@@ -274,4 +280,10 @@
             <inertia ixx="0.03" iyy="0.03" izz="0.03" ixy="0.0" ixz="0.0" iyz="0.0" />
         </inertial>
+        <collision>
+            <origin rpy="0 0 3.14159265359" xyz="0 0 0" />
+            <geometry>
+                <mesh filename="package://mecademic_description/meshes/finger.dae" />
+            </geometry>
+        </collision>
     </link>
     <joint name="meca_finger_joint1" type="prismatic">

Commit message: switching to effort

File: src/mecademic_description/urdf/meca_500_r3.urdf.xacro (robot description, xacro)
@@ -292,5 +292,5 @@
         <origin rpy="0 0 0" xyz="0 0 0.0584" />
         <axis xyz="0 1 0" />
-        <limit effort="20" lower="0.0" upper="0.04" velocity="0.2" />
+        <limit effort="9999" lower="-0.001" upper="0.06" velocity="0.1" />
     </joint>
     <joint name="meca_finger_joint2" type="prismatic">
@@ -299,5 +299,5 @@
         <origin rpy="0 0 0" xyz="0 0 0.0584" />
         <axis xyz="0 -1 0" />
-        <limit effort="20" lower="0.0" upper="0.04" velocity="0.2" />
+        <limit effort="9999" lower="-0.001" upper="0.06" velocity="0.1" />
         <mimic joint="meca_finger_joint1" />
     </joint>
@@ -365,8 +365,8 @@
         <type>transmission_interface/SimpleTransmission</type>
         <joint name="meca_finger_joint1">
-            <hardwareInterface>hardware_interface/PositionJointInterface</hardwareInterface>
+            <hardwareInterface>hardware_interface/EffortJointInterface</hardwareInterface>
         </joint>
         <actuator name="meca_finger_joint1_motor">
-            <hardwareInterface>hardware_interface/PositionJointInterface</hardwareInterface>
+            <hardwareInterface>hardware_interface/EffortJointInterface</hardwareInterface>
             <mechanicalReduction>1</mechanicalReduction>
         </actuator>
@@ -375,8 +375,8 @@
         <type>transmission_interface/SimpleTransmission</type>
         <joint name="meca_finger_joint2">
-            <hardwareInterface>hardware_interface/PositionJointInterface</hardwareInterface>
+            <hardwareInterface>hardware_interface/EffortJointInterface</hardwareInterface>
         </joint>
         <actuator name="meca_finger_joint2_motor">
-            <hardwareInterface>hardware_interface/PositionJointInterface</hardwareInterface>
+            <hardwareInterface>hardware_interface/EffortJointInterface</hardwareInterface>
             <mechanicalReduction>1</mechanicalReduction>
         </actuator>
@@ -394,3 +394,45 @@
         </plugin>
     </gazebo>
+    <gazebo reference="meca_rightfinger">
+        <mu1>100</mu1>
+        <mu2>100</mu2>
+        <kp>100000</kp>
+        <!-- <fdir1>0 0 0</fdir1> -->
+        <collision name="meca__leftfinger_collision">
+            <surface>
+                <friction>
+                    <torsional>
+                        <coefficient>100</coefficient>
+                        <use_patch_radius>true</use_patch_radius>
+                        <patch_radius>0.1</patch_radius>
+                        <surface_radius>0.1</surface_radius>
+                    </torsional>
+                </friction>
+            </surface>
+        </collision>
+    </gazebo>
+    <gazebo reference="meca_leftfinger">
+        <mu1>100</mu1>
+        <mu2>100</mu2>
+        <kp>100000</kp>
+        <!-- <fdir1>0 0 0</fdir1> -->
+        <collision name="meca__rightfinger_collision">
+            <surface>
+                <friction>
+                    <torsional>
+                        <coefficient>100</coefficient>
+                        <use_patch_radius>true</use_patch_radius>
+                        <patch_radius>0.1</patch_radius>
+                        <surface_radius>0.1</surface_radius>
+                    </torsional>
+                </friction>
+            </surface>
+        </collision>
+    </gazebo>
+    <!-- <gazebo reference="meca_finger_joint1">
+        <implicitSpringDamper>1</implicitSpringDamper>
+    </gazebo>
+    <gazebo reference="meca_finger_joint2">
+        <implicitSpringDamper>1</implicitSpringDamper>
+    </gazebo> -->
 </robot>

Commit message: inertia added but one finger missing

File: src/mecademic_description/urdf/meca_500_r3.urdf.xacro (robot description, xacro)
@@ -260,5 +260,6 @@
         <inertial>
             <mass value="0.1" />
-            <inertia ixx="0.03" iyy="0.03" izz="0.03" ixy="0.0" ixz="0.0" iyz="0.0" />
+            <origin xyz="0 0.0145644 0.0227941" rpy="0 0 0" />
+            <inertia ixx="3.01220925051e-05" ixy="0.0" ixz="0.0" iyy="2.95873808038e-05" iyz="0.0" izz="6.95125211657e-06" />
         </inertial>
         <collision>
@@ -278,5 +279,6 @@
         <inertial>
             <mass value="0.1" />
-            <inertia ixx="0.03" iyy="0.03" izz="0.03" ixy="0.0" ixz="0.0" iyz="0.0" />
+            <origin xyz="0 0.0145644 0.0227941" rpy="0 0 ${pi}" />
+            <inertia ixx="3.01220925051e-05" ixy="0.0" ixz="0.0" iyy="2.95873808038e-05" iyz="0.0" izz="6.95125211657e-06" />
         </inertial>
         <collision>
@@ -292,5 +294,5 @@
         <origin rpy="0 0 0" xyz="0 0 0.0584" />
         <axis xyz="0 1 0" />
-        <limit effort="9999" lower="-0.001" upper="0.06" velocity="0.1" />
+        <limit effort="1000" lower="-0.001" upper="0.04" velocity="0.3" />
     </joint>
     <joint name="meca_finger_joint2" type="prismatic">
@@ -299,5 +301,5 @@
         <origin rpy="0 0 0" xyz="0 0 0.0584" />
         <axis xyz="0 -1 0" />
-        <limit effort="9999" lower="-0.001" upper="0.06" velocity="0.1" />
+        <limit effort="1000" lower="-0.001" upper="0.04" velocity="0.3" />
         <mimic joint="meca_finger_joint1" />
     </joint>
@@ -399,5 +401,5 @@
         <kp>100000</kp>
         <!-- <fdir1>0 0 0</fdir1> -->
-        <collision name="meca__leftfinger_collision">
+        <collision name="meca_leftfinger_collision">
             <surface>
                 <friction>
@@ -417,5 +419,5 @@
         <kp>100000</kp>
         <!-- <fdir1>0 0 0</fdir1> -->
-        <collision name="meca__rightfinger_collision">
+        <collision name="meca_rightfinger_collision">
             <surface>
                 <friction>

Commit message: inertia fix

File: src/mecademic_description/urdf/meca_500_r3.urdf.xacro (robot description, xacro)
@@ -260,6 +260,7 @@
         <inertial>
             <mass value="0.1" />
-            <origin xyz="0 0.0145644 0.0227941" rpy="0 0 0" />
+            <!-- <origin xyz="0 0.0145644 0.0227941" rpy="0 0 0" /> -->
             <inertia ixx="3.01220925051e-05" ixy="0.0" ixz="0.0" iyy="2.95873808038e-05" iyz="0.0" izz="6.95125211657e-06" />
+            <!-- <inertia ixx="0.03" iyy="0.03" izz="0.03" ixy="0.0" ixz="0.0" iyz="0.0" /> -->
         </inertial>
         <collision>
@@ -279,6 +280,7 @@
         <inertial>
             <mass value="0.1" />
-            <origin xyz="0 0.0145644 0.0227941" rpy="0 0 ${pi}" />
+            <!-- <origin xyz="0 0.0145644 0.0227941" rpy="0 0 ${pi}" /> -->
             <inertia ixx="3.01220925051e-05" ixy="0.0" ixz="0.0" iyy="2.95873808038e-05" iyz="0.0" izz="6.95125211657e-06" />
+            <!-- <inertia ixx="0.03" iyy="0.03" izz="0.03" ixy="0.0" ixz="0.0" iyz="0.0" /> -->
         </inertial>
         <collision>
@@ -294,5 +296,5 @@
         <origin rpy="0 0 0" xyz="0 0 0.0584" />
         <axis xyz="0 1 0" />
-        <limit effort="1000" lower="-0.001" upper="0.04" velocity="0.3" />
+        <limit effort="99999" lower="-0.001" upper="0.04" velocity="0.3" />
     </joint>
     <joint name="meca_finger_joint2" type="prismatic">
@@ -301,5 +303,5 @@
         <origin rpy="0 0 0" xyz="0 0 0.0584" />
         <axis xyz="0 -1 0" />
-        <limit effort="1000" lower="-0.001" upper="0.04" velocity="0.3" />
+        <limit effort="99999" lower="-0.001" upper="0.04" velocity="0.3" />
         <mimic joint="meca_finger_joint1" />
     </joint>

Commit message: hand can pickup stuff thanks to the plugin bhttps://github.com/JenniferBuehler/gazebo-pkgs

File: src/mecademic_description/urdf/meca_500_r3.urdf.xacro (robot description, xacro)
@@ -217,34 +217,4 @@
             </geometry>
         </collision>
-        <!-- <collision>
-            <origin rpy="0 0 0" xyz="0 -0.05 0.04" />
-            <geometry>
-                <sphere radius="0.07" />
-            </geometry>
-        </collision>
-        <collision>
-            <origin rpy="0 0 0" xyz="0 0.05 0.04" />
-            <geometry>
-                <sphere radius="0.07" />
-            </geometry>
-        </collision> -->
-        <!-- <collision>
-            <origin rpy="0 1.57079632679 1.57079632679" xyz="0 0 0.1" />
-            <geometry>
-                <cylinder length="0.1" radius="0.05" />
-            </geometry>
-        </collision>
-        <collision>
-            <origin rpy="0 0 0" xyz="0 -0.05 0.1" />
-            <geometry>
-                <sphere radius="0.05" />
-            </geometry>
-        </collision>
-        <collision>
-            <origin rpy="0 0 0" xyz="0 0.05 0.1" />
-            <geometry>
-                <sphere radius="0.05" />
-            </geometry>
-        </collision> -->
         <inertial>
             <mass value="0.1" />
@@ -440,3 +410,20 @@
         <implicitSpringDamper>1</implicitSpringDamper>
     </gazebo> -->
+    <gazebo>
+        <plugin name="gazebo_grasp_fix" filename="libgazebo_grasp_fix.so">
+            <arm>
+                <arm_name>meca_arm</arm_name>
+                <palm_link>meca_axis_6_link</palm_link>
+                <gripper_link>meca_leftfinger</gripper_link>
+                <gripper_link> meca_rightfinger </gripper_link>
+            </arm>
+            <forces_angle_tolerance>100</forces_angle_tolerance>
+            <update_rate>4</update_rate>
+            <grip_count_threshold>4</grip_count_threshold>
+            <max_grip_count>8</max_grip_count>
+            <release_tolerance>0.005</release_tolerance>
+            <disable_collisions_on_attach>false</disable_collisions_on_attach>
+            <contact_topic>__default_topic__</contact_topic>
+        </plugin>
+    </gazebo>
 </robot>

Commit message: lowerd the efforts

File: src/mecademic_description/urdf/meca_500_r3.urdf.xacro (robot description, xacro)
@@ -266,5 +266,5 @@
         <origin rpy="0 0 0" xyz="0 0 0.0584" />
         <axis xyz="0 1 0" />
-        <limit effort="99999" lower="-0.001" upper="0.04" velocity="0.3" />
+        <limit effort="10" lower="-0.001" upper="0.04" velocity="0.3" />
     </joint>
     <joint name="meca_finger_joint2" type="prismatic">
@@ -273,5 +273,5 @@
         <origin rpy="0 0 0" xyz="0 0 0.0584" />
         <axis xyz="0 -1 0" />
-        <limit effort="99999" lower="-0.001" upper="0.04" velocity="0.3" />
+        <limit effort="10" lower="-0.001" upper="0.04" velocity="0.3" />
         <mimic joint="meca_finger_joint1" />
     </joint>

Commit message: added better looking bin

File: src/mecademic_description/urdf/meca_500_r3.urdf.xacro (robot description, xacro)
@@ -6,5 +6,5 @@
 <robot name="meca_500_r3">
     <!-- Base link is the center of the robot's bottom plate -->
-    <link name="world" />
+    <link name="world"/>
     <joint name="world_joint" type="fixed">
         <parent link="world" />

Commit message: added base to robot so it is detach from world

File: src/mecademic_description/urdf/meca_500_r3.urdf.xacro (robot description, xacro)
@@ -6,7 +6,21 @@
 <robot name="meca_500_r3">
     <!-- Base link is the center of the robot's bottom plate -->
-    <link name="world"/>
+    <link name="base_plate">
+        <visual>
+            <origin rpy="0 0 0" xyz="0 0 -0.005" />
+            <geometry>
+                <box size="0.1 0.1 0.01" />
+            </geometry>
+            <material name="white">
+                <color rgba="1 1.0 1.0 1.0" />
+            </material>
+        </visual>
+        <inertial>
+            <mass value="1000" />
+            <inertia ixx="0.03" ixy="0.0" ixz="0.0" iyy="0.03" iyz="0.0" izz="0.03" />
+        </inertial>
+    </link>
     <joint name="world_joint" type="fixed">
-        <parent link="world" />
+        <parent link="base_plate" />
         <child link="meca_base_link" />
         <origin rpy="0.0 0.0 0.0" xyz="0.0 0.0 0.0" />

Commit message: removed base plates and fix the robot to the world

File: src/mecademic_description/urdf/meca_500_r3.urdf.xacro (robot description, xacro)
@@ -6,5 +6,5 @@
 <robot name="meca_500_r3">
     <!-- Base link is the center of the robot's bottom plate -->
-    <link name="base_plate">
+    <!-- <link name="base_plate">
         <visual>
             <origin rpy="0 0 0" xyz="0 0 -0.005" />
@@ -20,7 +20,8 @@
             <inertia ixx="0.03" ixy="0.0" ixz="0.0" iyy="0.03" iyz="0.0" izz="0.03" />
         </inertial>
-    </link>
+    </link> -->
+    <link name="world" />
     <joint name="world_joint" type="fixed">
-        <parent link="base_plate" />
+        <parent link="world" />
         <child link="meca_base_link" />
         <origin rpy="0.0 0.0 0.0" xyz="0.0 0.0 0.0" />

Commit message: increased rotation angle for the joint 1 and added more effort to finger joint

File: src/mecademic_description/urdf/meca_500_r3.urdf.xacro (robot description, xacro)
@@ -69,5 +69,5 @@
         <child link="meca_axis_1_link" />
         <axis xyz="0 0 1" />
-        <limit effort="10.0" lower="-3.05433" upper="3.05433" velocity="2.61799" />
+        <limit effort="10.0" lower="-3.14141812" upper="3.14141812" velocity="2.61799" />
     </joint>
     <!-- Joint 2 -->
@@ -281,5 +281,5 @@
         <origin rpy="0 0 0" xyz="0 0 0.0584" />
         <axis xyz="0 1 0" />
-        <limit effort="10" lower="-0.001" upper="0.04" velocity="0.3" />
+        <limit effort="100" lower="-0.001" upper="0.04" velocity="0.3" />
     </joint>
     <joint name="meca_finger_joint2" type="prismatic">
@@ -288,5 +288,5 @@
         <origin rpy="0 0 0" xyz="0 0 0.0584" />
         <axis xyz="0 -1 0" />
-        <limit effort="10" lower="-0.001" upper="0.04" velocity="0.3" />
+        <limit effort="100" lower="-0.001" upper="0.04" velocity="0.3" />
         <mimic joint="meca_finger_joint1" />
     </joint>

Commit message: increased efforts

File: src/mecademic_description/urdf/meca_500_r3.urdf.xacro (robot description, xacro)
@@ -69,5 +69,5 @@
         <child link="meca_axis_1_link" />
         <axis xyz="0 0 1" />
-        <limit effort="10.0" lower="-3.14141812" upper="3.14141812" velocity="2.61799" />
+        <limit effort="100.0" lower="-3.14141812" upper="3.14141812" velocity="2.61799" />
     </joint>
     <!-- Joint 2 -->
@@ -95,5 +95,5 @@
         <child link="meca_axis_2_link" />
         <axis xyz="0 1 0" />
-        <limit effort="10.0" lower="-1.22173048" upper="1.5708" velocity="2.61799" />
+        <limit effort="100.0" lower="-1.22173048" upper="1.5708" velocity="2.61799" />
     </joint>
     <!-- Joint 3 -->
@@ -121,5 +121,5 @@
         <child link="meca_axis_3_link" />
         <axis xyz="0 1 0" />
-        <limit effort="10.0" lower="-2.35619" upper="1.22173048" velocity="3.14159" />
+        <limit effort="100.0" lower="-2.35619" upper="1.22173048" velocity="3.14159" />
     </joint>
     <!-- Joint 4 -->
@@ -147,5 +147,5 @@
         <child link="meca_axis_4_link" />
         <axis xyz="1 0 0" />
-        <limit effort="10.0" lower="-2.96706" upper="2.96706" velocity="5.23599" />
+        <limit effort="100.0" lower="-2.96706" upper="2.96706" velocity="5.23599" />
     </joint>
     <!-- Joint 5 -->
@@ -173,5 +173,5 @@
         <child link="meca_axis_5_link" />
         <axis xyz="0 1 0" />
-        <limit effort="10.0" lower="-2.00713" upper="2.00713" velocity="5.23599" />
+        <limit effort="100.0" lower="-2.00713" upper="2.00713" velocity="5.23599" />
     </joint>
     <!-- Joint 6 -->
@@ -199,5 +199,5 @@
         <child link="meca_axis_6_link" />
         <axis xyz="1 0 0" />
-        <limit effort="10.0" lower="-3.14159" upper="3.14159" velocity="8.72665" />
+        <limit effort="100.0" lower="-3.14159" upper="3.14159" velocity="8.72665" />
     </joint>
     <!-- <link name="meca_axis_flange" /> -->

Commit message: Revert "increased efforts"
This reverts commit bed0e26221d23c992dc7ea98fa9fecac004bbc79.

File: src/mecademic_description/urdf/meca_500_r3.urdf.xacro (robot description, xacro)
@@ -69,5 +69,5 @@
         <child link="meca_axis_1_link" />
         <axis xyz="0 0 1" />
-        <limit effort="100.0" lower="-3.14141812" upper="3.14141812" velocity="2.61799" />
+        <limit effort="10.0" lower="-3.14141812" upper="3.14141812" velocity="2.61799" />
     </joint>
     <!-- Joint 2 -->
@@ -95,5 +95,5 @@
         <child link="meca_axis_2_link" />
         <axis xyz="0 1 0" />
-        <limit effort="100.0" lower="-1.22173048" upper="1.5708" velocity="2.61799" />
+        <limit effort="10.0" lower="-1.22173048" upper="1.5708" velocity="2.61799" />
     </joint>
     <!-- Joint 3 -->
@@ -121,5 +121,5 @@
         <child link="meca_axis_3_link" />
         <axis xyz="0 1 0" />
-        <limit effort="100.0" lower="-2.35619" upper="1.22173048" velocity="3.14159" />
+        <limit effort="10.0" lower="-2.35619" upper="1.22173048" velocity="3.14159" />
     </joint>
     <!-- Joint 4 -->
@@ -147,5 +147,5 @@
         <child link="meca_axis_4_link" />
         <axis xyz="1 0 0" />
-        <limit effort="100.0" lower="-2.96706" upper="2.96706" velocity="5.23599" />
+        <limit effort="10.0" lower="-2.96706" upper="2.96706" velocity="5.23599" />
     </joint>
     <!-- Joint 5 -->
@@ -173,5 +173,5 @@
         <child link="meca_axis_5_link" />
         <axis xyz="0 1 0" />
-        <limit effort="100.0" lower="-2.00713" upper="2.00713" velocity="5.23599" />
+        <limit effort="10.0" lower="-2.00713" upper="2.00713" velocity="5.23599" />
     </joint>
     <!-- Joint 6 -->
@@ -199,5 +199,5 @@
         <child link="meca_axis_6_link" />
         <axis xyz="1 0 0" />
-        <limit effort="100.0" lower="-3.14159" upper="3.14159" velocity="8.72665" />
+        <limit effort="10.0" lower="-3.14159" upper="3.14159" velocity="8.72665" />
     </joint>
     <!-- <link name="meca_axis_flange" /> -->

Commit message: velocity changes

File: src/mecademic_description/urdf/meca_500_r3.urdf.xacro (robot description, xacro)
@@ -69,5 +69,5 @@
         <child link="meca_axis_1_link" />
         <axis xyz="0 0 1" />
-        <limit effort="10.0" lower="-3.14141812" upper="3.14141812" velocity="2.61799" />
+        <limit effort="10.0" lower="-3" upper="3" velocity="2" />
     </joint>
     <!-- Joint 2 -->
@@ -199,5 +199,5 @@
         <child link="meca_axis_6_link" />
         <axis xyz="1 0 0" />
-        <limit effort="10.0" lower="-3.14159" upper="3.14159" velocity="8.72665" />
+        <limit effort="10.0" lower="-3.14159" upper="3.14159" velocity="5.72665" />
     </joint>
     <!-- <link name="meca_axis_flange" /> -->
@@ -281,5 +281,5 @@
         <origin rpy="0 0 0" xyz="0 0 0.0584" />
         <axis xyz="0 1 0" />
-        <limit effort="100" lower="-0.001" upper="0.04" velocity="0.3" />
+        <limit effort="100" lower="-0.001" upper="0.04" velocity="0.1" />
     </joint>
     <joint name="meca_finger_joint2" type="prismatic">
@@ -288,5 +288,5 @@
         <origin rpy="0 0 0" xyz="0 0 0.0584" />
         <axis xyz="0 -1 0" />
-        <limit effort="100" lower="-0.001" upper="0.04" velocity="0.3" />
+        <limit effort="100" lower="-0.001" upper="0.04" velocity="0.1" />
         <mimic joint="meca_finger_joint1" />
     </joint>

Commit message: fixes (IDK)

File: src/mecademic_description/urdf/meca_500_r3.urdf.xacro (robot description, xacro)
@@ -69,5 +69,5 @@
         <child link="meca_axis_1_link" />
         <axis xyz="0 0 1" />
-        <limit effort="10.0" lower="-3" upper="3" velocity="2" />
+        <limit effort="10.0" lower="-3.05433" upper="3.05433" velocity="2.61799" />
     </joint>
     <!-- Joint 2 -->

Commit message: more improvements to make the robots run correctly

File: src/mecademic_description/urdf/meca_500_r3.urdf.xacro (robot description, xacro)
@@ -22,8 +22,8 @@
     </link> -->
     <link name="world" />
-    <joint name="world_joint" type="fixed">
+    <joint name="fixed" type="fixed">
         <parent link="world" />
         <child link="meca_base_link" />
-        <origin rpy="0.0 0.0 0.0" xyz="0.0 0.0 0.0" />
+        <!-- <origin rpy="0.0 0.0 0.0" xyz="0.0 0.0 0.0" /> -->
     </joint>
     <link name="meca_base_link">
