Commit message: increased effort and planner change

File: src/mecademic_description/urdf/meca_500_r3.urdf.xacro (robot description, xacro)
@@ -69,5 +69,5 @@
         <child link="meca_axis_1_link" />
         <axis xyz="0 0 1" />
-        <limit effort="10.0" lower="-3.05433" upper="3.05433" velocity="2.61799" />
+        <limit effort="1000.0" lower="-3.05433" upper="3.05433" velocity="2.61799" />
     </joint>
     <!-- Joint 2 -->
@@ -95,5 +95,5 @@
         <child link="meca_axis_2_link" />
         <axis xyz="0 1 0" />
-        <limit effort="10.0" lower="-1.22173048" upper="1.5708" velocity="2.61799" />
+        <limit effort="1000.0" lower="-1.22173048" upper="1.5708" velocity="2.61799" />
     </joint>
     <!-- Joint 3 -->
@@ -121,5 +121,5 @@
         <child link="meca_axis_3_link" />
         <axis xyz="0 1 0" />
-        <limit effort="10.0" lower="-2.35619" upper="1.22173048" velocity="3.14159" />
+        <limit effort="1000.0" lower="-2.35619" upper="1.22173048" velocity="3.14159" />
     </joint>
     <!-- Joint 4 -->
@@ -147,5 +147,5 @@
         <child link="meca_axis_4_link" />
         <axis xyz="1 0 0" />
-        <limit effort="10.0" lower="-2.96706" upper="2.96706" velocity="5.23599" />
+        <limit effort="1000.0" lower="-2.96706" upper="2.96706" velocity="5.23599" />
     </joint>
     <!-- Joint 5 -->
@@ -173,5 +173,5 @@
         <child link="meca_axis_5_link" />
         <axis xyz="0 1 0" />
-        <limit effort="10.0" lower="-2.00713" upper="2.00713" velocity="5.23599" />
+        <limit effort="1000.0" lower="-2.00713" upper="2.00713" velocity="5.23599" />
     </joint>
     <!-- Joint 6 -->
@@ -199,5 +199,5 @@
         <child link="meca_axis_6_link" />
         <axis xyz="1 0 0" />
-        <limit effort="10.0" lower="-3.14159" upper="3.14159" velocity="5.72665" />
+        <limit effort="1000.0" lower="-3.14159" upper="3.14159" velocity="5.72665" />
     </joint>
     <!-- <link name="meca_axis_flange" /> -->
